File: led_matrix/v1/led_mat_v1/led_mat_v1.kicad_sch (KiCad schematic)
At the start: 124 parts, among them J1 Left_header, J2 Right_header

Commit message: feat(led_matrix): add PCB/schematic exports and update KiCad project files
- Add 3D PCB view export (led_mat_v1.png) and schematic export (led_mat_v1.svg)
- Update schematic, PCB layout, and project files with latest design changes
- Exclude KiCad lock files (*.lck) from version control via .gitignore
Other:
- note added: "ARDUINO NANO"
- note added: "LED MATRIX"
- note added: "PIN HEADERS"
- company: (none) -> Misbah Ali Mir
- title: (none) -> Charlieplexing LED Matrix
- moved on the sheet: A1, D1,10, D1,11, D1,2, D1,3, D1,4, D1,5, D1,6, D1,7, D1,8, D1,9, D10,1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
